File: PCB/Puntodroid-ADAS/puntodroid-adas/puntodroid-adas.kicad_sch (KiCad schematic)
At the start: 0 parts

Commit message: update puntodroid schematic
Other:
- added sheet CAN INTERFACE (pundodroid-adas-can.kicad_sch)
- added sheet POWER (puntodroid-power.kicad_sch)
- added sheet RADIO RFM69 (puntodroid-radio.kicad_sch)
Changed lines of the file:
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@@
+	)
+	(sheet
+		(at 117.475 78.105)
+		(size 35.56 26.035)
+		(exclude_from_sim no)
+		(in_bom yes)
+		(on_board yes)
+		(dnp no)
+		(fields_autoplaced yes)
+		(stroke
+			(width 0.1524)
+			(type solid)
+		)
+		(fill
+			(color 0 0 0 0.0000)
+		)
+		(property "Sheetname" "POWER"
+			(at 117.475 77.3934 0)
+			(effects
+				(font
+					(size 1.27 1.27)
+				)
+				(justify left bottom)
+			)
+		)
+		(property "Sheetfile" "puntodroid-power.kicad_sch"
+			(at 117.475 104.7246 0)
+			(effects
+				(font
+					(size 1.27 1.27)
+				)
+				(justify left top)
+			)
+		)
+		(instances
+			(project "puntodroid-adas"
+				(path "/427bbe6b-ed35-4841-963c-5b19708bc81b"
+					(page "5")
+				)
+			)
+		)
+	)
+	(sheet
+		(at 53.975 78.105)
+		(size 35.56 26.035)
+		(exclude_from_sim no)
+		(in_bom yes)
+		(on_board yes)
+		(dnp no)
+		(fields_autoplaced yes)
+		(stroke
+			(width 0.1524)
+			(type solid)
+		)
+		(fill
+			(color 0 0 0 0.0000)
+		)
+		(property "Sheetname" "CAN INTERFACE"
+			(at 53.975 77.3934 0)
+			(effects
+				(font
+					(size 1.27 1.27)
+				)
+				(justify left bottom)
+			)
+		)
+		(property "Sheetfile" "pundodroid-adas-can.kicad_sch"
+			(at 53.975 104.7246 0)
+			(effects
+				(font
+					(size 1.27 1.27)
+				)
+				(justify left top)
+			)
+		)
+		(instances
+			(project "puntodroid-adas"
+				(path "/427bbe6b-ed35-4841-963c-5b19708bc81b"
+					(page "4")
+				)
+			)
+		)
 	)
 	(sheet
@@
 				)
 			)
+		)
+	)
+	(sheet
+		(at 53.975 113.03)
+		(size 35.56 23.495)
+		(exclude_from_sim no)
+		(in_bom yes)
+		(on_board yes)
+		(dnp no)
+		(fields_autoplaced yes)
+		(stroke
+			(width 0.1524)
+			(type solid)
+		)
+		(fill
+			(color 0 0 0 0.0000)
+		)
+		(property "Sheetname" "RADIO RFM69"
+			(at 53.975 112.3184 0)
+			(effects
+				(font
+					(size 1.27 1.27)
+				)
+				(justify left bottom)
+			)
+		)
+		(property "Sheetfile" "puntodroid-radio.kicad_sch"
+			(at 53.975 137.1096 0)
+			(effects
+				(font
+					(size 1.27 1.27)
+				)
+				(justify left top)
+			)
+		)
+		(instances
+			(project "puntodroid-adas"
+				(path "/427bbe6b-ed35-4841-963c-5b19708bc81b"
+					(page "6")
+				)
+			)

Commit message: update puntodroid schematic stm32
Other:
- added sheet CONNECTORS (puntodroid-connectors.kicad_sch)
Changed lines of the file:
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@@
+	)
+	(sheet
+		(at 116.84 115.062)
+		(size 35.56 23.876)
+		(exclude_from_sim no)
+		(in_bom yes)
+		(on_board yes)
+		(dnp no)
+		(fields_autoplaced yes)
+		(stroke
+			(width 0.1524)
+			(type solid)
+		)
+		(fill
+			(color 0 0 0 0.0000)
+		)
+		(property "Sheetname" "CONNECTORS"
+			(at 116.84 114.3504 0)
+			(effects
+				(font
+					(size 1.27 1.27)
+				)
+				(justify left bottom)
+			)
+		)
+		(property "Sheetfile" "puntodroid-connectors.kicad_sch"
+			(at 116.84 139.5226 0)
+			(effects
+				(font
+					(size 1.27 1.27)
+				)
+				(justify left top)
+			)
+		)
+		(instances
+			(project "puntodroid-adas"
+				(path "/427bbe6b-ed35-4841-963c-5b19708bc81b"
+					(page "7")
+				)
+			)
+		)
 	)
 	(sheet
