File: PCB/Puntodroid-ADAS/puntodroid-adas/puntodroid-adas.kicad_sch (KiCad schematic)
At the start: 0 parts

Commit message: move to kicad v10. change rfm69 to lora radio, add push button connector, add puntodroid logo
Other:
- sheet RADIO RFM69 renamed RADIO RA-02 LORA
- added sheet CAR DISTANCE SENSOR (puntodroid-distance-sensor.kicad_sch)
- added sheet PUSH_BUTTONS (puntodroid-push-buttons.kicad_sch)
Changed lines of the file:
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@@
 (kicad_sch
-	(version 20250114)
+	(version 20260306)
 	(generator "eeschema")
-	(generator_version "9.0")
+	(generator_version "10.0")
 	(paper "A4")
 	(sheet
@@
 		)
 		(fill
-			(color 0 0 0 0.0000)
+			(color 0 0 0 0)
 		)
 		(property "Sheetname" "STM32F microcontroller"
 			(at 53.975 35.4834 0)
+			(show_name no)
+			(do_not_autoplace no)
 			(effects
 				(font
@@
 		(property "Sheetfile" "puntodroid-adas-stm32.kicad_sch"
 			(at 53.975 65.3546 0)
+			(show_name no)
+			(do_not_autoplace no)
 			(effects
 				(font
@@
 		)
 		(fill
-			(color 0 0 0 0.0000)
+			(color 0 0 0 0)
 		)
 		(property "Sheetname" "POWER"
 			(at 117.475 77.3934 0)
+			(show_name no)
+			(do_not_autoplace no)
 			(effects
 				(font
@@
 		(property "Sheetfile" "puntodroid-power.kicad_sch"
 			(at 117.475 104.7246 0)
+			(show_name no)
+			(do_not_autoplace no)
 			(effects
 				(font
@@
 		)
 		(fill
-			(color 0 0 0 0.0000)
+			(color 0 0 0 0)
 		)
 		(property "Sheetname" "CONNECTORS"
 			(at 116.84 114.3504 0)
+			(show_name no)
+			(do_not_autoplace no)
 			(effects
 				(font
@@
 		(property "Sheetfile" "puntodroid-connectors.kicad_sch"
 			(at 116.84 139.5226 0)
+			(show_name no)
+			(do_not_autoplace no)
 			(effects
 				(font
@@
 				(path "/427bbe6b-ed35-4841-963c-5b19708bc81b"
 					(page "7")
+				)
+			)
+		)
+	)
+	(sheet
+		(at 116.84 147.32)
+		(size 35.56 25.4)
+		(exclude_from_sim no)
+		(in_bom yes)
+		(on_board yes)
+		(dnp no)
+		(fields_autoplaced yes)
+		(stroke
+			(width 0.1524)
+			(type solid)
+		)
+		(fill
+			(color 0 0 0 0)
+		)
+		(property "Sheetname" "PUSH_BUTTONS"
+			(at 116.84 146.6084 0)
+			(show_name no)
+			(do_not_autoplace no)
+			(effects
+				(font
+					(size 1.27 1.27)
+				)
+				(justify left bottom)
+			)
+		)
+		(property "Sheetfile" "puntodroid-push-buttons.kicad_sch"
+			(at 116.84 173.3046 0)
+			(show_name no)
+			(do_not_autoplace no)
+			(effects
+				(font
+					(size 1.27 1.27)
+				)
+				(justify left top)
+			)
+		)
+		(instances
+			(project "puntodroid-adas"
+				(path "/427bbe6b-ed35-4841-963c-5b19708bc81b"
+					(page "9")
 				)
 			)
@@
 		)
 		(fill
-			(color 0 0 0 0.0000)
+			(color 0 0 0 0)
 		)
 		(property "Sheetname" "CAN INTERFACE"
 			(at 53.975 77.3934 0)
+			(show_name no)
+			(do_not_autoplace no)
 			(effects
 				(font
@@
 		(property "Sheetfile" "pundodroid-adas-can.kicad_sch"
 			(at 53.975 104.7246 0)
+			(show_name no)
+			(do_not_autoplace no)
 			(effects
 				(font
@@
 		)
 		(fill
-			(color 0 0 0 0.0000)
+			(color 0 0 0 0)
 		)
 		(property "Sheetname" "CAMERA"
 			(at 117.475 35.4834 0)
+			(show_name no)
+			(do_not_autoplace no)
 			(effects
 				(font
@@
 		(property "Sheetfile" "puntodroid-adas-camera.kicad_sch"
 			(at 117.475 65.3546 0)
+			(show_name no)
+			(do_not_autoplace no)
 			(effects
 				(font
@@
 				(path "/427bbe6b-ed35-4841-963c-5b19708bc81b"
 					(page "3")
+				)
+			)
+		)
+	)
+	(sheet
+		(at 54.61 147.32)
+		(size 34.29 26.67)
+		(exclude_from_sim no)
+		(in_bom yes)
+		(on_board yes)
+		(dnp no)
+		(fields_autoplaced yes)
+		(stroke
+			(width 0.1524)
+			(type solid)
+		)
+		(fill
+			(color 0 0 0 0)
+		)
+		(property "Sheetname" "CAR DISTANCE SENSOR"
+			(at 54.61 146.6084 0)
+			(show_name no)
+			(do_not_autoplace no)
+			(effects
+				(font
+					(size 1.27 1.27)
+				)
+				(justify left bottom)
+			)
+		)
+		(property "Sheetfile" "puntodroid-distance-sensor.kicad_sch"
+			(at 54.61 174.5746 0)
+			(show_name no)
+			(do_not_autoplace no)
+			(effects
+				(font
+					(size 1.27 1.27)
+				)
+				(justify left top)
+			)
+		)
+		(instances
+			(project "puntodroid-adas"
+				(path "/427bbe6b-ed35-4841-963c-5b19708bc81b"
+					(page "8")
 				)
 			)
@@
 		)
 		(fill
-			(color 0 0 0 0.0000)
-		)
-		(property "Sheetname" "RADIO RFM69"
+			(color 0 0 0 0)
+		)
+		(property "Sheetname" "RADIO RA-02 LORA"
 			(at 53.975 112.3184 0)
+			(show_name no)
+			(do_not_autoplace no)
 			(effects
 				(font
@@
 		(property "Sheetfile" "puntodroid-radio.kicad_sch"
 			(at 53.975 137.1096 0)
-			(effects
-				(font
+			(show_name no)
+			(do_not_autoplace no)
+			(effects
+				(font
