File: PCB/Puntodroid-ADAS/puntodroid-adas/pundodroid-adas-can.kicad_sch (KiCad schematic)
At the start: 12 parts, among them U6 SN65HVD230, U7 TJA1054

Commit message: update puntodroid schematic stm32
Parts:
- added J8: FIAT_OBD2_SOCKET, symbol Connector_Generic:Conn_02x08_Top_Bottom
- added J9: PUNTO_CAN, symbol Connector_Generic:Conn_01x04
Connections:
- net CANH_HS_CAR: now also J8.6 (Pin_6), J9.1 (Pin_1)
- net CANH_LS_CAR: now also J8.1 (Pin_1), J9.3 (Pin_3)
- net CANL_HS_CAR: now also J8.14 (Pin_14), J9.2 (Pin_2)
- net CANL_LS_CAR: now also J8.9 (Pin_9), J9.4 (Pin_4)
- new net POWER_GND: J8.4 (Pin_4)
- new net SIGNAL_GND: J8.5 (Pin_5)
- new net VBAT_12V: J8.16 (Pin_16)
Other:
- note added: "CAN CONNECTOR CONNECT TO OBD2 SOCKET"
- note added: "OBD2 PINOUT (NOT ON THE BOARD)"

Commit message: add quick charger
Parts:
- C21: renamed from C20; footprint (none) -> Capacitor_SMD:C_0805_2012Metric_Pad1.18x1.45mm_HandSolder
- C22: renamed from C19; footprint (none) -> Capacitor_SMD:C_0805_2012Metric_Pad1.18x1.45mm_HandSolder
- R20: renamed from R17; footprint (none) -> Resistor_SMD:R_0805_2012Metric_Pad1.20x1.40mm_HandSolder
- R21: renamed from R16; footprint (none) -> Resistor_SMD:R_0805_2012Metric_Pad1.20x1.40mm_HandSolder
- R22: renamed from R18; footprint (none) -> Resistor_SMD:R_0805_2012Metric_Pad1.20x1.40mm_HandSolder
- R23: renamed from R19; footprint (none) -> Resistor_SMD:R_0805_2012Metric_Pad1.20x1.40mm_HandSolder
- U7: footprint (none) -> Package_SO:SO-14_3.9x8.65mm_P1.27mm
- renumbered D2 to D1, D1 to D2, J8 to J7, J9 to J8
Changed lines of the file:
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@@
 		(dnp no)
 		(fields_autoplaced yes)
-		(property "Reference" "#PWR034"
+		(property "Reference" "#PWR049"
 			(at 78.74 127 0)
 			(effects
@@
 			(project "puntodroid-adas"
 				(path "/427bbe6b-ed35-4841-963c-5b19708bc81b/8fb622c5-2309-48f8-8ec8-1b99fc8c9e6b"
-					(reference "#PWR034")
+					(reference "#PWR049")
 					(unit 1)
 				)
@@
 			)
 		)
-		(property "Footprint" ""
+		(property "Footprint" "Package_SO:SO-14_3.9x8.65mm_P1.27mm"
 			(at 71.12 143.51 0)
 			(effects
@@
 		(on_board yes)
 		(dnp no)
-		(property "Reference" "R16"
+		(property "Reference" "R21"
 			(at 73.406 107.188 0)
 			(effects
@@
 			)
 		)
-		(property "Footprint" ""
+		(property "Footprint" "Resistor_SMD:R_0805_2012Metric_Pad1.20x1.40mm_HandSolder"
 			(at 71.628 107.95 90)
 			(effects
@@
 			(project "puntodroid-adas"
 				(path "/427bbe6b-ed35-4841-963c-5b19708bc81b/8fb622c5-2309-48f8-8ec8-1b99fc8c9e6b"
-					(reference "R16")
+					(reference "R21")
 					(unit 1)
 				)
@@
 		(dnp no)
 		(fields_autoplaced yes)
-		(property "Reference" "#PWR038"
+		(property "Reference" "#PWR048"
 			(at 78.74 46.99 0)
 			(effects
@@
 			(project "puntodroid-adas"
 				(path "/427bbe6b-ed35-4841-963c-5b19708bc81b/8fb622c5-2309-48f8-8ec8-1b99fc8c9e6b"
-					(reference "#PWR038")
+					(reference "#PWR048")
 					(unit 1)
 				)
@@
 		(on_board no)
 		(dnp no)
-		(property "Reference" "J8"
+		(property "Reference" "J7"
 			(at 169.164 53.086 0)
 			(effects
@@
 			(project ""
 				(path "/427bbe6b-ed35-4841-963c-5b19708bc81b/8fb622c5-2309-48f8-8ec8-1b99fc8c9e6b"
-					(reference "J8")
+					(reference "J7")
 					(unit 1)
 				)
@@
 		(dnp no)
 		(fields_autoplaced yes)
-		(property "Reference" "#PWR033"
+		(property "Reference" "#PWR047"
 			(at 72.39 172.72 0)
 			(effects
@@
 			(project "puntodroid-adas"
 				(path "/427bbe6b-ed35-4841-963c-5b19708bc81b/8fb622c5-2309-48f8-8ec8-1b99fc8c9e6b"
-					(reference "#PWR033")
+					(reference "#PWR047")
 					(unit 1)
 				)
@@
 		(on_board yes)
 		(dnp no)
-		(property "Reference" "C19"
+		(property "Reference" "C22"
 			(at 83.566 116.078 0)
 			(effects
@@
 			)
 		)
-		(property "Footprint" ""
+		(property "Footprint" "Capacitor_SMD:C_0805_2012Metric_Pad1.18x1.45mm_HandSolder"
 			(at 77.7748 113.03 0)
 			(effects
@@
 			(project "puntodroid-adas"
 				(path "/427bbe6b-ed35-4841-963c-5b19708bc81b/8fb622c5-2309-48f8-8ec8-1b99fc8c9e6b"
-					(reference "C19")
+					(reference "C22")
 					(unit 1)
 				)
@@
 		(on_board yes)
 		(dnp no)
-		(property "Reference" "C20"
+		(property "Reference" "C21"
 			(at 83.566 36.068 0)
 			(effects
@@
 			)
 		)
-		(property "Footprint" ""
+		(property "Footprint" "Capacitor_SMD:C_0805_2012Metric_Pad1.18x1.45mm_HandSolder"
 			(at 77.7748 33.02 0)
 			(effects
@@
 			(project "puntodroid-adas"
 				(path "/427bbe6b-ed35-4841-963c-5b19708bc81b/8fb622c5-2309-48f8-8ec8-1b99fc8c9e6b"
-					(reference "C20")
+					(reference "C21")
 					(unit 1)
 				)
@@
 		(dnp no)
 		(fields_autoplaced yes)
-		(property "Reference" "#PWR036"
+		(property "Reference" "#PWR044"
 			(at 69.85 30.48 0)
 			(effects
@@
 			(project "puntodroid-adas"
 				(path "/427bbe6b-ed35-4841-963c-5b19708bc81b/8fb622c5-2309-48f8-8ec8-1b99fc8c9e6b"
-					(reference "#PWR036")
+					(reference "#PWR044")
 					(unit 1)
 				)
@@
 		(dnp no)
 		(fields_autoplaced yes)
-		(property "Reference" "J9"
+		(property "Reference" "J8"
 			(at 185.42 109.2199 0)
 			(effects
@@
 			(project ""
 				(path "/427bbe6b-ed35-4841-963c-5b19708bc81b/8fb622c5-2309-48f8-8ec8-1b99fc8c9e6b"
-					(reference "J9")
+					(reference "J8")
 					(unit 1)
 				)
@@
 		(on_board yes)
 		(dnp no)
-		(property "Reference" "R18"
+		(property "Reference" "R22"
 			(at 90.17 148.59 90)
 			(effects
@@
 			)
 		)
-		(property "Footprint" ""
+		(property "Footprint" "Resistor_SMD:R_0805_2012Metric_Pad1.20x1.40mm_HandSolder"
 			(at 90.17 144.272 90)
 			(effects
@@
 			(project "puntodroid-adas"
 				(path "/427bbe6b-ed35-4841-963c-5b19708bc81b/8fb622c5-2309-48f8-8ec8-1b99fc8c9e6b"
-					(reference "R18")
+					(reference "R22")
 					(unit 1)
 				)
@@
 		(on_board yes)
 		(dnp no)
-		(property "Reference" "D1"
+		(property "Reference" "D2"
 			(at 92.202 64.77 90)
 			(effects
@@
 			(project ""
 				(path "/427bbe6b-ed35-4841-963c-5b19708bc81b/8fb622c5-2309-48f8-8ec8-1b99fc8c9e6b"
-					(reference "D1")
+					(reference "D2")
 					(unit 1)
 				)
@@
 		(on_board yes)
 		(dnp no)
-		(property "Reference" "R19"
+		(property "Reference" "R23"
 			(at 102.616 138.938 90)
 			(effects
@@
 			)
 		)
-		(property "Footprint" ""
+		(property "Footprint" "Resistor_SMD:R_0805_2012Metric_Pad1.20x1.40mm_HandSolder"
 			(at 102.87 141.732 90)
 			(effects
@@
 			(project "puntodroid-adas"
 				(path "/427bbe6b-ed35-4841-963c-5b19708bc81b/8fb622c5-2309-48f8-8ec8-1b99fc8c9e6b"
-					(reference "R19")
+					(reference "R23")
 					(unit 1)
 				)
@@
 		(on_board yes)
 		(dnp no)
-		(property "Reference" "D2"
+		(property "Reference" "D1"
 			(at 84.328 64.77 90)
 			(effects
@@
 			(project "puntodroid-adas"
 				(path "/427bbe6b-ed35-4841-963c-5b19708bc81b/8fb622c5-2309-48f8-8ec8-1b99fc8c9e6b"
-					(reference "D2")
+					(reference "D1")
 					(unit 1)
 				)
@@
 		(dnp no)
 		(fields_autoplaced yes)
-		(property "Reference" "#PWR035"
+		(property "Reference" "#PWR043"
 			(at 50.8 124.46 0)
 			(effects
@@
 			(project "puntodroid-adas"
 				(path "/427bbe6b-ed35-4841-963c-5b19708bc81b/8fb622c5-2309-48f8-8ec8-1b99fc8c9e6b"
-					(reference "#PWR035")
+					(reference "#PWR043")
 					(unit 1)
 				)
@@
 		(dnp no)
 		(fields_autoplaced yes)
-		(property "Reference" "#PWR032"
+		(property "Reference" "#PWR046"
 			(at 69.85 106.68 0)
 			(effects
@@
 			(project ""
 				(path "/427bbe6b-ed35-4841-963c-5b19708bc81b/8fb622c5-2309-48f8-8ec8-1b99fc8c9e6b"
-					(reference "#PWR032")
+					(reference "#PWR046")
 					(unit 1)
 				)
@@
 		(on_board yes)
 		(dnp no)
-		(property "Reference" "R17"
+		(property "Reference" "R20"
 			(at 45.974 128.778 0)
 			(effects
@@
 			)
 		)
-		(property "Footprint" ""
+		(property "Footprint" "Resistor_SMD:R_0805_2012Metric_Pad1.20x1.40mm_HandSolder"
 			(at 52.578 129.54 90)
 			(effects
@@
 			(project "puntodroid-adas"
 				(path "/427bbe6b-ed35-4841-963c-5b19708bc81b/8fb622c5-2309-48f8-8ec8-1b99fc8c9e6b"
-					(reference "R17")
+					(reference "R20")
 					(unit 1)
 				)
@@
 		(dnp no)
 		(fields_autoplaced yes)
-		(property "Reference" "#PWR037"
+		(property "Reference" "#PWR045"
 			(at 69.85 82.55 0)
 			(effects
@@
 			(project "puntodroid-adas"
 				(path "/427bbe6b-ed35-4841-963c-5b19708bc81b/8fb622c5-2309-48f8-8ec8-1b99fc8c9e6b"
-					(reference "#PWR037")
-					(unit 1)
-				)
+					(reference "#PWR045")
+					(unit 1)
+				)
