File: PCB/Puntodroid-ADAS/puntodroid-adas/puntodroid-adas-camera.kicad_sch (KiCad schematic)
At the start: 0 parts

Commit message: update camera video path
Parts:
- added C11: 100u, symbol Device:C_Polarized_Small
- added C14: 22u, symbol Device:C_Polarized_Small
- added C15, C16, C17, C18: 100n, symbol Device:C
- added FB1, FB2, FB3: FerriteBead, symbol Device:FerriteBead_Small
- added J4: RCA_SOCKET, symbol Connector:Conn_Coaxial_x2
- added J5: VIDEO_OUTPUT, symbol Connector:Conn_Coaxial
- added NT2: VIDEO_GND_NETTIE, symbol Device:NetTie_3_Tee
- added R10, R15, R6, R7, R8, R9: 0R, symbol Device:R
- added R11: 10k, symbol Device:R
- added R12, R13, R14: 75R, symbol Device:R
- added U3: AT7456, symbol My-Lib:AT7456
- added U4: PI5V330, symbol My-Lib:PI5V330
- added U5: THS7373, Package_SO:TSSOP-14_4.4x5mm_P0.65mm, symbol My-Lib:THS7373
- added Y2: 27MHz, symbol Device:Crystal
Connections:
- new net: C11.1, C14.1, R12.1
- new net: C11.2, R10.2, U3.26 (VOUT)
- new net: U3.1 (NC), U3.15 (NC)
- new net: U3.13 (NC), U3.27 (NC)
- new net: U3.14 (NC), U3.28 (NC)
- new net: U3.16 (NC), U3.2 (NC)
- new net: R11.1, U3.18 (~{HSYNC})
- new net: FB1.1, U3.21 (AVDD)
- new net: C15.1, R10.1, U3.22 (VIN)
- new net: C14.2, U3.25 (SAG)
- new net: U3.5 (CLKIN), Y2.2
- new net: U3.6 (XFB), Y2.1
- new net: R9.1, U5.13 (HD_CH1_OUT)
- new net: C15.2, R13.2, R8.2, R9.2
- new net: R14.2, R6.1, R7.1, U4.4 (D_{A})
- new net: J4.1 (IN1), U4.2 (S1A)
- new net: J4.2 (IN2), U4.3 (S2A)
- new net: R15.2, R8.1, U5.14 (CVBS_OUT)
- new net: J5.1 (In), R12.2
- new net: R15.1, R6.2, U5.1 (CVBS_IN)
- new net: FB3.2, NT2.1
- new net: R7.2, U5.2 (HD_CH1_IN)
- new net: FB2.2, NT2.2
- new net +5V: FB1.2, R11.2, U3.24 (PVDD), U3.3 (DVDD), U4.16 (VCC), U5.10 (VCC)
- new net AT7456_CS: U3.8 (~{CS})
- new net AT7456_LOS: U3.12 (LOS)
- new net AT7456_RESET: U3.19 (~{RESET})
- new net AT7456_SCK: U3.10 (SDCLK)
- new net AT7456_SDIN: U3.9 (SDIN)
- new net AT7456_SDOUT: U3.11 (SDOUT)
- new net AT7456_VSYNC: U3.17 (~{VSYNC})
- new net GNDD: NT2.3, U3.4 (DGND), U4.15 (~{EN}), U4.8 (GND), U5.5 (GND), U5.6 (DISABLE)
- new net GNDP: U3.23 (PGND)
- new net GNDV: FB2.1, FB3.1, J4.3 (EXT), J5.2 (Ext), R13.1, R14.1, U3.20 (AGND)
- new net HD_BYPASS: U5.9 (HD_BYPASS)
- new net VIDEO_MUX: U4.1 (IN)
- no-connect marks 0 -> 12
Other:
- note added: "AT7456 BTYPASS"
- note added: "BYPASS: HIGH: ON LOW: OFF"
- note added: "CVBS/HD INPUT SELECT"
- note added: "CVBS/HD OUTPUT SELECT"
- note added: "IN LOW: S1X IN HIGH: S2X"
- note added: "THS7373 BTYPASS"

Commit message: update puntodroid schematic
Parts:
- added J6: CAMERA POWER SUPPLY, symbol Connector_Generic:Conn_01x04
- added Q1, Q3: AO3401A, Package_TO_SOT_SMD:SOT-23, symbol Transistor_FET:AO3401A
- added Q2, Q4: BC817, Package_TO_SOT_SMD:SOT-23, symbol Transistor_BJT:BC817
- added R23, R25: 47k, symbol Device:R
- added R24, R26: 10k, symbol Device:R
Connections:
- net GNDD: now also Q2.2 (E), Q4.2 (E)
- net GNDP: now also J6.1 (Pin_1), J6.3 (Pin_3)
- new net: Q2.1 (B), R24.2
- new net: Q1.1 (G), Q2.3 (C), R23.1
- new net: J6.4 (Pin_4), Q1.3 (D)
- new net: J6.2 (Pin_2), Q3.3 (D)
- new net: Q4.1 (B), R26.2
- new net: Q3.1 (G), Q4.3 (C), R25.1
- new net +12V: Q1.2 (S), Q3.2 (S), R23.2, R25.2
- new net CAMERA_BACK_EN: R26.1
- new net CAMERA_FRONT_EN: R24.1
Other:
- note added: "VIDEO BUFFER"
- note added: "VIDEO MUX"
- note added: "VIDEO OSD"
- moved on the sheet: C11, C14, C15, C16, C17, C18, FB1, FB2, FB3, J4, J5, NT2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

Commit message: update puntodroid schematic stm32
Connections:
- net +5V: now also C16.1, C17.1, C18.1
- net GNDD: now also C16.2
- net GNDP: now also C17.2
- net GNDV: now also C18.2
Other:
- note added: "CAMERA POWER ENABLE"
- moved on the sheet: C15, C16, C17, C18, J5, Q2, Q3, Q4, R12, R23, R24, R25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

Commit message: add quick charger
Parts:
- removed FB2: FerriteBead, symbol Device:FerriteBead_Small
- removed NT2: VIDEO_GND_NETTIE, symbol Device:NetTie_3_Tee
- added C13, C14: 100n, Capacitor_SMD:C_0805_2012Metric_Pad1.18x1.45mm_HandSolder, symbol Device:C
- added NT1: VIDEO_GND_NETTIE, My-Footprints:NetTie-2x, symbol Device:NetTie_2
- C15: footprint (none) -> Capacitor_SMD:C_0805_2012Metric_Pad1.18x1.45mm_HandSolder
- C16: renamed from C17; footprint (none) -> Capacitor_SMD:C_0805_2012Metric_Pad1.18x1.45mm_HandSolder
- C17: renamed from C18; footprint (none) -> Capacitor_SMD:C_0805_2012Metric_Pad1.18x1.45mm_HandSolder
- C18: renamed from C16; footprint (none) -> Capacitor_SMD:C_0805_2012Metric_Pad1.18x1.45mm_HandSolder
- C19: renamed from C14; footprint (none) -> Capacitor_THT:CP_Radial_D6.3mm_P2.50mm
- C20: renamed from C11; footprint (none) -> Capacitor_THT:CP_Radial_D6.3mm_P2.50mm
- R10: renamed from R7; footprint (none) -> Resistor_SMD:R_0805_2012Metric_Pad1.20x1.40mm_HandSolder
- R11: renamed from R25; footprint (none) -> Resistor_SMD:R_0805_2012Metric_Pad1.20x1.40mm_HandSolder
- R12: renamed from R26; footprint (none) -> Resistor_SMD:R_0805_2012Metric_Pad1.20x1.40mm_HandSolder
- R13: renamed from R15; footprint (none) -> Resistor_SMD:R_0805_2012Metric_Pad1.20x1.40mm_HandSolder
- R14: renamed from R8; footprint (none) -> Resistor_SMD:R_0805_2012Metric_Pad1.20x1.40mm_HandSolder
- R15: renamed from R9; footprint (none) -> Resistor_SMD:R_0805_2012Metric_Pad1.20x1.40mm_HandSolder
- R16: renamed from R13; footprint (none) -> Resistor_SMD:R_0805_2012Metric_Pad1.20x1.40mm_HandSolder
- R17: renamed from R11; footprint (none) -> Resistor_SMD:R_0805_2012Metric_Pad1.20x1.40mm_HandSolder
- R18: renamed from R10; footprint (none) -> Resistor_SMD:R_0805_2012Metric_Pad1.20x1.40mm_HandSolder
- R19: renamed from R12; footprint (none) -> Resistor_SMD:R_0805_2012Metric_Pad1.20x1.40mm_HandSolder
- R6: renamed from R23; footprint (none) -> Resistor_SMD:R_0805_2012Metric_Pad1.20x1.40mm_HandSolder
- R7: renamed from R24; footprint (none) -> Resistor_SMD:R_0805_2012Metric_Pad1.20x1.40mm_HandSolder
- R8: renamed from R14; footprint (none) -> Resistor_SMD:R_0805_2012Metric_Pad1.20x1.40mm_HandSolder
- R9: renamed from R6; footprint (none) -> Resistor_SMD:R_0805_2012Metric_Pad1.20x1.40mm_HandSolder
- U3: renamed from U4; footprint (none) -> Package_SO:SOIC-16_3.9x9.9mm_P1.27mm
- U5: renamed from U3; footprint (none) -> Package_SO:TSSOP-28_4.4x9.7mm_P0.65mm
- renumbered FB3 to FB1, FB1 to FB2, J6 to J4, J4 to J5, J5 to J6, U5 to U4
Connections:
- net +5V: now also C13.2, C14.2
- net GNDD: now also C13.1, C14.1, NT1.2
- net at FB1.2: now also NT1.1
Other:
- moved on the sheet: FB1
