File: PCB/Puntodroid-ADAS/puntodroid-adas/puntodroid-connectors.kicad_sch (KiCad schematic)
At the start: 8 parts, among them J10 DS18B20, J7 UNUSED_PINS, Q5 BC817

Commit message: add quick charger
Parts:
- J16: renamed from J10; footprint (none) -> My-Footprints-connectors:JST_XH_B3B-XH-A_1x03_P2.50mm_Vertical
- J17: renamed from J7; footprint (none) -> My-Footprints-connectors:PinHeader_2x20_P2.54mm_Vertical
- renumbered D6 to D8, Q5 to Q9, R27 to R35, R28 to R36, R29 to R37
Connections:
- net +3.3V: now also J17.19 (Pin_19)
Other:
- moved on the sheet: R35
