File: PCB/Puntodroid-ADAS/puntodroid-adas/puntodroid-power.kicad_sch (KiCad schematic)
At the start: 13 parts, among them U8 MP1584-Step-Down, U9 AMS1117

Commit message: update puntodroid schematic stm32
Parts:
- added D8, D9: BZV55B3V3, Diode_SMD:D_MiniMELF, symbol Diode:BZV55B5V6
- added J12: V_BAT_12V, symbol Connector_Generic:Conn_01x02
- added J13: ANDROID_RADIO, symbol Connector_Generic:Conn_01x04
- added Q6: AO3401A, Package_TO_SOT_SMD:SOT-23, symbol Transistor_FET:AO3401A
- added Q7, Q9: BC817, Package_TO_SOT_SMD:SOT-23, symbol Transistor_BJT:BC817
- added Q8: BC807, Package_TO_SOT_SMD:SOT-23, symbol Transistor_BJT:BC807
- added R30, R36: 47k, symbol Device:R
- added R31, R37: 10k, symbol Device:R
- added R32: 30k, Resistor_SMD:R_0805_2012Metric_Pad1.20x1.40mm_HandSolder, symbol Device:R
- added R33: 2k7, Resistor_SMD:R_0805_2012Metric_Pad1.20x1.40mm_HandSolder, symbol Device:R
- added R34: 22k, Resistor_SMD:R_0805_2012Metric_Pad1.20x1.40mm_HandSolder, symbol Device:R
- added R35: 5k6, Resistor_SMD:R_0805_2012Metric_Pad1.20x1.40mm_HandSolder, symbol Device:R
- C21: value C_Polarized -> 1000u/25V
- F1: value Fuse -> 3A
Connections:
- net +12V: now also J13.2 (Pin_2), Q6.2 (S), Q8.2 (E), R30.2, R36.2
- net +5V: now also R34.1
- net GNDD: now also D8.2 (A), D9.2 (A), Q7.2 (E), Q9.2 (E), R33.2, R35.2
- net GNDP: now also J13.3 (Pin_3)
- net at D5.2 (A), F1.2: now also R32.1
- net VBAT_NEG: no longer names the net of FL1.2
- net VBAT_NEG: now also J12.1 (Pin_1)
- net VBAT_POS: no longer names the net of F1.1
- net VBAT_POS: now also J12.2 (Pin_2)
- new net: Q6.1 (G), Q7.3 (C), R36.1
- new net: J13.1 (Pin_1), Q6.3 (D)
- new net: J13.4 (Pin_4), Q8.3 (C)
- new net: Q7.1 (B), R37.2
- new net: Q9.1 (B), R31.2
- new net: Q8.1 (B), Q9.3 (C), R30.1
- new net ADC_5V: D9.1 (K), R34.2, R35.1
- new net ADC_VBATT_12V: D8.1 (K), R32.2, R33.1
- new net ANDROID_EN: R37.1
- new net REVERSE_SIGNAL: R31.1
Other:
- note added: "+12V BATT"
- note added: "12V ADC INPUT"
- note added: "5V ADC INPUT"
- note added: "ANDROID RADIO POWER"
- note added: "IGNITION"
- note added: "REVERSE"
- moved on the sheet: C21, C22, C23, C24, C25, D5, F1, FL1, R20, R21, R22, U8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

Commit message: add quick charger
Parts:
- added C28: 100n, Capacitor_SMD:C_0805_2012Metric_Pad1.18x1.45mm_HandSolder, symbol Device:C
- added C29, C30: 1u, Capacitor_SMD:C_0805_2012Metric_Pad1.18x1.45mm_HandSolder, symbol Device:C
- added J10: USB_A_Stacked, symbol Connector:USB_A_Stacked
- added J12, J13: POWER_12V, symbol Connector_Generic:Conn_01x02
- added J14, J15: POWER_5V, symbol Connector_Generic:Conn_01x02
- added MOD1: QUICK_CHARGER, My-Footprints:Quick_Charger_ SW3518, symbol My-Lib:Quick_Charger_USB
- added NT2: NetTie_2, My-Footprints:NetTie-2x, symbol Device:NetTie_2
- C27: renamed from C21; footprint (none) -> Capacitor_THT:CP_Radial_D10.0mm_P3.80mm
- F1: footprint (none) -> My-Footprints:Fuseholder_Clip-5x20mm_Eaton_1A5601-01_Inline_P20.80x6.76mm_D1.70mm_Horizontal
- R31: renamed from R36; footprint (none) -> Resistor_SMD:R_0805_2012Metric_Pad1.20x1.40mm_HandSolder
- R32: renamed from R37; footprint (none) -> Resistor_SMD:R_0805_2012Metric_Pad1.20x1.40mm_HandSolder
- R33: renamed from R30; footprint (none) -> Resistor_SMD:R_0805_2012Metric_Pad1.20x1.40mm_HandSolder
- R34: renamed from R31; footprint (none) -> Resistor_SMD:R_0805_2012Metric_Pad1.20x1.40mm_HandSolder
- U8: footprint (none) -> My-Footprints-converters-modules:MP1584_Mini_3A_Step_Down_Conv
- renumbered C22 to C23, C23 to C24, C24 to C25, C25 to C26, D8 to D6, D9 to D7, J13 to J11, J12 to J9, Q6 to Q5, Q7 to Q6, Q8 to Q7, Q9 to Q8, R20 to R24, R21 to R25, R22 to R26, R32 to R27, R33 to R28, R34 to R29, R35 to R30
Connections:
- net +12V: now also C28.1, J12.2 (Pin_2), J13.2 (Pin_2), MOD1.2 (VCC)
- net +5V: now also C29.1, C30.1, J10.1 (VBUS1), J10.5 (VBUS2), J14.2 (Pin_2), J15.2 (Pin_2)
- net GNDD: now also NT2.2
- net GNDP: now also C28.2, C29.2, C30.2, J10.4 (GND1), J10.8 (GND2), J10.9 (Shield), J12.1 (Pin_1), J13.1 (Pin_1), J14.1 (Pin_1), J15.1 (Pin_1), MOD1.1 (GND), NT2.1
- new net: J10.2 (D1-), J10.6 (D2-)
- new net: J10.3 (D1+), J10.7 (D2+)
Other:
- note added: "GND NETTIE"
- note added: "POWER CONNECTORS"
- note added: "USB SOCKETS"
