File: PCB/Puntodroid-ADAS/puntodroid-adas/puntodroid-radio.kicad_sch (KiCad schematic)
At the start: 0 parts

Commit message: update puntodroid schematic stm32
Parts:
- added AE1: Antenna, symbol Device:Antenna
- added C26: 100n, symbol Device:C
- added U11: RFM69HCW, symbol RF_Module:RFM69HCW
Connections:
- new net: AE1.1 (A), U11.9 (ANT)
- new net +3.3V: C26.2, U11.13 (3.3V)
- new net GNDD: C26.1, U11.1 (GND), U11.10 (GND), U11.8 (GND)
- new net RFM69_CS: U11.5 (NSS)
- new net RFM69_MISO: U11.2 (MISO)
- new net RFM69_MOSI: U11.3 (MOSI)
- new net RFM69_RESET: U11.6 (RESET)
- new net RFM69_SCK: U11.4 (SCK)
Other:
- note added: "RFM69 RADIO MODULE"

Commit message: add quick charger
Parts:
- AE1: footprint (none) -> Capacitor_SMD:C_0805_2012Metric_Pad1.18x1.45mm_HandSolder
- C31: renamed from C26; footprint (none) -> Capacitor_SMD:C_0805_2012Metric_Pad1.18x1.45mm_HandSolder
- U10: renamed from U11; footprint (none) -> RF_Module:HOPERF_RFM69HW
Changed lines of the file:
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@@
 		(on_board yes)
 		(dnp no)
-		(property "Reference" "#PWR061"
+		(property "Reference" "#PWR085"
 			(at 54.61 43.18 0)
 			(effects
@@
 			(project "puntodroid-adas"
 				(path "/427bbe6b-ed35-4841-963c-5b19708bc81b/c7f6453c-9930-4ee9-995f-ac357768c1b9"
-					(reference "#PWR061")
+					(reference "#PWR085")
 					(unit 1)
 				)
@@
 		(on_board yes)
 		(dnp no)
-		(property "Reference" "C26"
+		(property "Reference" "C31"
 			(at 49.784 32.258 0)
 			(effects
@@
 			)
 		)
-		(property "Footprint" ""
+		(property "Footprint" "Capacitor_SMD:C_0805_2012Metric_Pad1.18x1.45mm_HandSolder"
 			(at 55.5752 29.21 0)
 			(effects
@@
 			(project "puntodroid-adas"
 				(path "/427bbe6b-ed35-4841-963c-5b19708bc81b/c7f6453c-9930-4ee9-995f-ac357768c1b9"
-					(reference "C26")
+					(reference "C31")
 					(unit 1)
 				)
@@
 		(dnp no)
 		(fields_autoplaced yes)
-		(property "Reference" "U11"
+		(property "Reference" "U10"
 			(at 65.6433 39.37 0)
 			(effects
@@
 			)
 		)
-		(property "Footprint" ""
+		(property "Footprint" "RF_Module:HOPERF_RFM69HW"
 			(at -20.32 12.7 0)
 			(effects
@@
 			(project ""
 				(path "/427bbe6b-ed35-4841-963c-5b19708bc81b/c7f6453c-9930-4ee9-995f-ac357768c1b9"
-					(reference "U11")
+					(reference "U10")
 					(unit 1)
 				)
@@
 			)
 		)
-		(property "Footprint" ""
+		(property "Footprint" "Capacitor_SMD:C_0805_2012Metric_Pad1.18x1.45mm_HandSolder"
 			(at 85.09 33.02 0)
 			(effects
@@
 		(dnp no)
 		(fields_autoplaced yes)
-		(property "Reference" "#PWR059"
+		(property "Reference" "#PWR087"
 			(at 66.04 78.74 0)
 			(effects
@@
 			(project "puntodroid-adas"
 				(path "/427bbe6b-ed35-4841-963c-5b19708bc81b/c7f6453c-9930-4ee9-995f-ac357768c1b9"
-					(reference "#PWR059")
+					(reference "#PWR087")
 					(unit 1)
 				)
@@
 		(dnp no)
 		(fields_autoplaced yes)
-		(property "Reference" "#PWR060"
+		(property "Reference" "#PWR086"
 			(at 63.5 31.75 0)
 			(effects
@@
 			(project "puntodroid-adas"
 				(path "/427bbe6b-ed35-4841-963c-5b19708bc81b/c7f6453c-9930-4ee9-995f-ac357768c1b9"
-					(reference "#PWR060")
-					(unit 1)
-				)
+					(reference "#PWR086")
+					(unit 1)
+				)
